File: V1.0/RP_LM2596-KfzPowerSafeguard.kicad_pcb (KiCad board)
At the start: 2 copper layers, 61 x 40.6 mm, 37 parts, among them J1 Conn_02x03_Odd_Even, J2 Conn_02x03_Odd_Even, J3 Conn_02x03_Odd_Even, Q1 BSP613P, Q10 TSM7P06, Q2 BSP613P, Q20 TSM7P06, U1 YAAJ_DCDC_StepDown_LM2596, X1 Faston 6.3, X2 Faston 6.3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

Commit message: V1.0 Product datat generated
10 pcs orderd at JLCPCB.com
Other:
- rule pad_to_mask_clearance: 0.051 -> 0
